File: Telemetry_pcb/Data collection pcb/Data collection pcb.kicad_pcb (KiCad board)
At the start: 2 copper layers, 18 parts, among them U1 HELTEC V4 LORA, U2 ADC_MODULE, U3 ACCELEROMETER, U4 GPS_MODULE, U5 VOLTAGE_DIVIDER, U6 VOLTAGE_DIVIDER

Commit message: idkidkidkidkidkidk
Parts:
- moved 3.3V_RAIL_1 27.4 mm to (199.0, 129.2)
- moved ESC_PADS_1 27.4 mm to (131.2, 131.2)
- moved GND_RAIL_1 27.4 mm to (199.0, 83.6)
- moved SCL_RAIL_1 27.4 mm to (94.9, 120.7)
- moved SPARE_GPIO_PADS_1 27.4 mm to (147.4, 50.8)
- moved U1 27.4 mm to (130.1, 109.0)
- moved U5 27.4 mm to (160.1, 121.6)
- moved U6 27.4 mm to (180.1, 121.6)
- moved 5V_RAIL_1 27.4 mm to (163.5, 66.8)
- moved U3 27.4 mm to (164.7, 86.8)
- moved U4 27.4 mm to (99.6, 89.3)
- moved BATTERY_VOLTAGE_PADS_1 27.4 mm to (163.7, 130.8)
- moved CURRENT_SENSOR_PADS_1 27.4 mm to (144.9, 131.3)
- moved MOTOR_VOLTAGE_PADS_1 27.4 mm to (184.5, 130.8)
- moved RPM_SENSOR_PADS_1 27.4 mm to (112.9, 131.3)
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Connections:
- net /3.3 renamed +3.3V
- net /5V renamed +5V
- net /GND renamed GND
Routing:
- net +3.3V: track 0.00 -> 248.9 mm, vias 0 -> 3
- net GND: track 0.00 -> 234.4 mm, vias 0 -> 3
- net /SCL: track 0.00 -> 147.9 mm, vias 0 -> 2
- net /SDA: track 0.00 -> 139.6 mm, vias 0 -> 2
- net +5V: track 0.00 -> 135.4 mm, vias 0 -> 2
- net /TEMP: track 0.00 -> 96.8 mm, vias 0 -> 2
- net /MOTV: track 0.00 -> 87.3 mm
- net /GPSTX: track 0.00 -> 74.2 mm, vias 0 -> 1
- net /GPSRX: track 0.00 -> 74.1 mm, vias 0 -> 1
- net /BATV: track 0.00 -> 65.1 mm
- net /CVREF: track 0.00 -> 64.5 mm, vias 0 -> 1
- net /WRPM: track 0.00 -> 63.9 mm, vias 0 -> 1
- net /MRPM: track 0.00 -> 60.8 mm, vias 0 -> 1
- net /CVOUT: track 0.00 -> 59.7 mm
- net /GP37: track 0.00 -> 57.7 mm, vias 0 -> 1
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Other:
- board outline added: 120 x 100 mm

Commit message: finished data collection pcb
Parts:
- added H1: MountingHole, MountingHole:MountingHole_3.2mm_M3, F.Cu at (94.0, 44.0)
- added H2: MountingHole, MountingHole:MountingHole_3.2mm_M3, F.Cu at (190.0, 55.0)
- added H3: MountingHole, MountingHole:MountingHole_3.2mm_M3, F.Cu at (204.0, 134.0)
- added H4: MountingHole, MountingHole:MountingHole_3.2mm_M3, F.Cu at (94.0, 134.0)
Routing:
- net GND: track 234.4 -> 67.0 mm, vias 3 -> 0
- net +5V: track 135.4 -> 242.4 mm
- net +3.3V: track 248.9 -> 319.2 mm, vias 3 -> 2
- added copper zone on F.Cu, net GND
Other:
- outline, holes or cut-outs redrawn
- board text added: "ASCTE Greenpower Data Collection"

Commit message: added sd and rtc to pcb
Parts:
- added U7: SD_BOARD, telem_system_footprint_library:SD_BOARD, F.Cu at (94.5, 56.4)
- added U8: RTC_MODULE, telem_system_footprint_library:RTC_MODULE, F.Cu at (92.7, 118.5)
- moved H1 23.0 mm to (71.0, 44.0)
- moved H4 23.0 mm to (71.0, 134.0)
Routing:
- net /GP7: track 19.5 -> 180.7 mm
- net /GP47: track 32.8 -> 142.9 mm
- net /GP48: track 29.2 -> 116.8 mm
- net /SDA: track 139.6 -> 225.3 mm, vias 2 -> 4
- net GND: track 67.0 -> 142.2 mm, vias 0 -> 5
- net /SCL: track 147.9 -> 221.2 mm, vias 2 -> 3
- net /GP5: track 23.5 -> 75.0 mm
- net +3.3V: track 319.2 -> 358.9 mm
Other:
- board size 120 x 100 mm -> 143 x 100 mm
- board text added: "RTC_MODULE"
- board text added: "SD_BOARD"
